File: SPROJ3G2_Receiver_PCB.kicad_sch (KiCad schematic)
At the start: 55 parts, among them J1 2137160001, J2 UART_Con, J3 SWDIO_Con, J4 Servo_Con, J5 7V_Supply_Voltage_Con, J6 3V3_Supply_Voltage_Con, J7 RF24_Con, Q1 ZXMN3A03E6TA, U1 RP2040, U2 W25Q128JVSIQ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

Commit message: Schematic cleanup
Schematic cleanup
Other:
- note added: "12MHz Crystal Oscillator"
- note added: "2MB SPI Flash"
- note added: "Boot button"
- note added: "nRF24L01 connector"
- note removed: "16MB SPI Flash Chip"
- note removed: "Boot mode button"
- note removed: "Crystal Oscillator"
- note removed: "RF24 connector"
- company: SDU Sonderborg -> SDU Sønderborg
- title: SPROJ3G2 - Receiver Logic PCB -> SPROJ3EEG2 - PRX PCB
Changed lines of the file:
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@@
 	(paper "A4")
 	(title_block
-		(title "SPROJ3G2 - Receiver Logic PCB")
-		(date "2024-11-11")
-		(rev "1.1")
-		(company "SDU Sonderborg")
-		(comment 1 "Author: Bence Toth")
+		(title "SPROJ3EEG2 - PRX PCB")
+		(date "2024-12-20")
+		(rev "1.3")
+		(company "SDU Sønderborg")
+		(comment 1 "Author: Bence Tóth")
 	)
 	(junction
@@
 		)
 	)
-	(text "Boot mode button"
+	(text "Boot button"
 		(exclude_from_sim no)
-		(at 102.87 28.194 0)
+		(at 102.362 27.686 0)
 		(effects
 			(font
 				(face "KiCad Font")
-				(size 1.84 1.84)
+				(size 2 2)
 				(thickness 0.368)
 				(bold yes)
-				(italic yes)
 			)
 		)
@@
 			(font
 				(face "KiCad Font")
-				(size 1.84 1.84)
+				(size 2 2)
 				(thickness 0.368)
 				(bold yes)
-				(italic yes)
 			)
 		)
@@
 			(font
 				(face "KiCad Font")
-				(size 1.84 1.84)
+				(size 2 2)
 				(thickness 0.368)
 				(bold yes)
-				(italic yes)
 			)
 		)
@@
 			(font
 				(face "KiCad Font")
-				(size 1.84 1.84)
+				(size 2 2)
 				(thickness 0.368)
 				(bold yes)
-				(italic yes)
 			)
 		)
@@
 	(text "Raspberry Pi RP2040 MCU"
 		(exclude_from_sim no)
-		(at 221.742 23.368 0)
+		(at 221.488 22.098 0)
 		(effects
 			(font
 				(face "KiCad Font")
-				(size 1.84 1.84)
+				(size 2 2)
 				(thickness 0.368)
 				(bold yes)
-				(italic yes)
 			)
 		)
 	)
-	(text "RF24 connector"
+	(text "nRF24L01 connector"
 		(exclude_from_sim no)
 		(at 84.836 74.93 0)
@@
 			(font
 				(face "KiCad Font")
-				(size 1.84 1.84)
+				(size 2 2)
 				(thickness 0.368)
 				(bold yes)
-				(italic yes)
 			)
 		)
 	)
-	(text "16MB SPI Flash Chip"
+	(text "2MB SPI Flash"
 		(exclude_from_sim no)
 		(at 51.816 17.272 0)
@@
 			(font
 				(face "KiCad Font")
-				(size 1.84 1.84)
+				(size 2 2)
 				(thickness 0.368)
 				(bold yes)
-				(italic yes)
 			)
 		)
@@
 	(text "Reset button"
 		(exclude_from_sim no)
-		(at 141.224 18.288 0)
+		(at 147.32 21.082 0)
 		(effects
 			(font
 				(face "KiCad Font")
-				(size 1.84 1.84)
+				(size 2 2)
 				(thickness 0.368)
 				(bold yes)
-				(italic yes)
 			)
 		)
@@
 	(text "Power Supply selector"
 		(exclude_from_sim no)
-		(at 28.702 161.544 0)
+		(at 29.464 161.544 0)
 		(effects
 			(font
 				(face "KiCad Font")
-				(size 1.84 1.84)
+				(size 2 2)
 				(thickness 0.368)
 				(bold yes)
-				(italic yes)
 			)
 		)
@@
 			(font
 				(face "KiCad Font")
-				(size 1.84 1.84)
+				(size 2 2)
 				(thickness 0.368)
 				(bold yes)
-				(italic yes)
 			)
 		)
 	)
-	(text "Crystal Oscillator"
+	(text "12MHz Crystal Oscillator"
 		(exclude_from_sim no)
 		(at 156.21 77.47 0)
@@
 			(font
 				(face "KiCad Font")
-				(size 1.84 1.84)
+				(size 2 2)
 				(thickness 0.368)
 				(bold yes)
-				(italic yes)
 			)
 		)
@@
 			(font
 				(face "KiCad Font")
-				(size 1.84 1.84)
+				(size 2 2)
 				(thickness 0.368)
 				(bold yes)
-				(italic yes)
 			)
 		)
@@
 		(on_board yes)
 		(dnp no)
-		(fields_autoplaced yes)
 		(property "Reference" "C1"
-			(at 17.78 31.7499 0)
+			(at 20.066 30.48 0)
 			(effects
 				(font
@@
 		)
 		(property "Value" "100n"
-			(at 17.78 34.2899 0)
+			(at 20.828 35.814 0)
 			(effects
 				(font
